File: lipo-psu.sch (KiCad schematic (older format))
At the start: 19 parts, among them J1 S4B-XH-A(LF)(SN), Q1 Si2301CDS, Q2 AO3400A, Q3 Si2301CDS, U1 BQ296100, U2 TPS7A2633DRVR

Commit message: changes
Parts:
- added H1, H2, H3, H4, H5, H6, H7, H8: MountingHole, MountingHole:MountingHole_2.5mm, symbol Mechanical:MountingHole
- added JP1: current_test, Jumper:SolderJumper-2_P1.3mm_Open_TrianglePad1.0x1.5mm, symbol Jumper:SolderJumper_2_Open
- added JP2: no_prot_opt, Jumper:SolderJumper-2_P1.3mm_Open_TrianglePad1.0x1.5mm, symbol Jumper:SolderJumper_2_Open
- C4: Digikey (none) -> 1276-2083-1-ND
- C6: Digikey (none) -> 1276-1291-1-ND
- J1: value S4B-XH-A(LF)(SN) -> 4Pin; footprint Connector_JST:JST_XH_S4B-XH-A_1x04_P2.50mm_Horizontal -> Connector_PinHeader_2.54mm:PinHeader_1x04_P2.54mm_Vertical; LCSC C157925 -> (none)
- Q1, Q3: Digikey (none) -> SI2301CDS-T1-GE3
- Q2: Alternative (none) -> PMV40UN2R‎; Digikey (none) -> 1727-1900-1-ND
- R3: Digikey (none) -> ‎RMCF0603FG100RCT-ND‎
- R4: Digikey (none) -> RNCP0603FTD4R70CT-ND
Connections:
- net +BATT: now also JP2.2 (B)
- net at Q3.2 (S), R3.1, R6.2: now also JP1.2 (B); no longer BT1.1 (+), R1.2
- new net: BT1.1 (+), JP1.1 (A), JP2.1 (A), R1.2
- no-connect marks 0 -> 1
Other:
- note added: "2 mA\nmax!"
- note added: "Connector"
- note removed: "https://www.digikey.de/short/znvbn9"
- moved on the sheet: BT1, C1, C2, C3, C4, C5, C6, J1, Q1, Q2, Q3, R1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
